Commit message: Xacro changes and ros2_control changes

File: src/rover/description/urdf/rover.ros2_control.xacro (robot description, xacro)
@@ -2,18 +2,18 @@
 <robot xmlns:xacro="http://www.ros.org/wiki/xacro">
   <!-- Copied from: https://github.com/ros-controls/ros2_control_demos/blob/master/example_2/description/ros2_control/diffbot.ros2_control.xacro -->
-  <xacro:macro name="diffbot_ros2_control" params="name use_mock_hardware">     <ros2_control name="${name}" type="system">
-      <xacro:unless value="${use_mock_hardware}">
-	<hardware>
+  <xacro:macro name="diffbot_ros2_control" params="name use_gazebo:=^|false">
+    <ros2_control name="${name}" type="system">
+      <hardware>
+	<xacro:if value="${use_gazebo}">
+	  <plugin>gz_ros2_control/GazeboSimSystem</plugin>
+	</xacro:if>
+	<xacro:unless value="${use_gazebo}">
+	  <!-- Replace this with my own hardware interfaces -->
 	  <plugin>ros2_control_demo_example_2/DiffBotSystemHardware</plugin>
 	  <param name="example_param_hw_start_duration_sec">0</param>
 	  <param name="example_param_hw_stop_duration_sec">3.0</param>
-	</hardware>
-      </xacro:unless>
-      <xacro:if value="${use_mock_hardware}">
-	<hardware>
-	  <plugin>mock_components/GenericSystem</plugin>
-	  <param name="calculate_dynamics">true</param>
-	</hardware>
-      </xacro:if>
+	  <param name="example_param_hw_slowdown">100</param> <!-- Unsure what this is for-->
+	</xacro:unless>
+      </hardware>
       <joint name="left_wheel_joint">
 	<command_interface name="velocity"/>
@@ -26,12 +26,11 @@
 	<state_interface name="velocity"/>
       </joint>
+      <joint name="caster_axis">
+        <state_interface name="position"/>
+      </joint>
+      <joint name="caster_wheel_joint">
+        <state_interface name="position"/>
+      </joint>
     </ros2_control>
   </xacro:macro>
-  <!-- plugin to parse tags and load interfaces -->
-  <gazebo>
-    <plugin filename="libgz_ros2_control-system.so" name="gz_ros2_control::GazeboSimROS2ControlPlugin">
-      <parameters>$(find rover)/config/robot_controllers.yaml</parameters>
-      <controller_manager_prefix_node_name>controller_manager</controller_manager_prefix_node_name>
-    </plugin>
-  </gazebo>
 </robot>

File: src/rover/description/urdf/rover.xacro (robot description, xacro)
@@ -1,7 +1,9 @@
 <?xml version="1.0"?>
 <robot xmlns:xacro="http://www.ros.org/wiki/xacro" name="robot">
-  <xacro:arg name="use_mock_hardware" default="false" />
+  <xacro:arg name="use_gazebo" default="false" />
   <xacro:include filename="rover_base.xacro"/>
   <xacro:include filename="rover.ros2_control.xacro"/>
-  <xacro:diffbot_ros2_control name="rover" use_mock_hardware="$(arg use_mock_hardware)"/>
+  <xacro:diffbot_ros2_control name="rover" use_gazebo="$(arg use_gazebo)"/>
+  <xacro:include filename="rover.gazebo.xacro"/>
+  <xacro:include filename="camera.xacro"/>
 </robot>

File: src/rover/description/urdf/rover_base.xacro (robot description, xacro)
@@ -5,5 +5,6 @@
 	<xacro:property name="tire_width" value="0.08"/>
 	<xacro:property name="axle_offset" value="0.055"/>
-	<xacro:property name="caster_offset" value="0.07"/>
+	<xacro:property name="caster_axis_offset" value="0.07"/>
+        <xacro:property name="caster_trail" value="0.045"/>
 	<xacro:property name="base_width" value="0.615"/>
 	<xacro:property name="base_length" value="1.22"/>
@@ -11,4 +12,7 @@
 	<xacro:property name="base_lift" value="0.305"/> <!--Distance between ground and center of base-->
 	<xacro:property name="PI" value="3.141592653"/>
+	<xacro:property name="wheel_mass" value="2"/>
+	<xacro:property name="wheel_friction" value="1.2"/>
+	<xacro:property name="base_mass" value="15"/>
 	<xacro:macro name="zero_origin">
 		<origin xyz='0 0 0' rpy='0 0 0'/>
@@ -20,13 +24,15 @@
 		<color rgba="0.1 0.1 0.1 1" />
 	</material>
-	<link name='world'/>
-	<joint name='world_to_chassis' type='fixed'>
-		<parent link = 'world'/>
-		<child link = 'chassis'/>
-		<origin xyz= '0 0 ${base_lift}' rpy='0 0 0'/>
+        <link name='base_link'>
+                <xacro:zero_origin/>
+        </link>
+	<joint name='base_to_chassis' type='fixed'>
+		<parent link='base_link'/>
+		<child link='chassis'/>
+		<origin xyz='-${base_length / 2 - axle_offset} 0 ${base_lift}' rpy='0 0 0'/>
 	</joint>
 	<link name='chassis'>
 		<visual>
-			<xacro:zero_origin/>
+                        <xacro:zero_origin/>
 			<geometry>
 				<box size="${base_length} ${base_width} ${base_thickness}"/>
@@ -35,5 +41,5 @@
 		</visual>
 		<collision>
-			<xacro:zero_origin/>
+                        <xacro:zero_origin/>
 			<geometry>
 				<box size="${base_length} ${base_width} ${base_thickness}"/>
@@ -41,9 +47,34 @@
 		</collision>
 		<inertial>
-			<xacro:zero_origin/>
-			<mass value="4.14395"/>
+                        <xacro:zero_origin/>
+			<mass value="${base_mass}"/>
 			<inertia ixx='0.1' ixy='0' ixz='0' iyy='0.2' iyz='0' izz='0.2'/>
 		</inertial>
 	</link>
+        <joint name="chassis_to_chungus" type="fixed">
+		<parent link='chassis'/>
+		<child link='chungus_mass'/>
+		<origin xyz='${base_length / 2 - axle_offset} 0 ${base_thickness / 2 + 0.1}' rpy='0 0 0'/>
+	</joint>
+        <link name="chungus_mass">
+		<visual>
+			<xacro:zero_origin/>
+			<geometry>
+				<box size="0.2 0.2 0.2"/>
+			</geometry>
+			<material name="black"/>
+		</visual>
+		<collision>
+			<xacro:zero_origin/>
+			<geometry>
+				<box size="0.2 0.2 0.2"/>
+			</geometry>
+		</collision>
+		<inertial>
+			<xacro:zero_origin/>
+			<mass value="10"/>
+			<inertia ixx='0.3' ixy='0' ixz='0' iyy='0.3' iyz='0' izz='0.3'/>
+		</inertial>
+        </link>
 	<!--TODO: NEEDS TO RUN ALONGSIDE JOINT_STATE_PUBLISHER-->
 	<!-- left wheel -->
@@ -67,8 +98,14 @@
 				<cylinder radius='${tire_diam / 2}' length='${tire_width}'/>
 			</geometry>
+                        <surface>
+                                <friction>
+                                        <mu>0.9</mu>
+                                        <mu2>0.9</mu2>
+                                </friction>
+                        </surface>
 		</collision>
 		<inertial>
 			<xacro:zero_origin/>
-			<mass value="0.5"/>
+			<mass value="${wheel_mass}"/>
 			<inertia ixx='0.3' ixy='0' ixz='0' iyy='0.3' iyz='0' izz='0.5'/>
 		</inertial>
@@ -93,35 +130,64 @@
 				<cylinder radius='${tire_diam / 2}' length='${tire_width}'/>
 			</geometry>
+                        <surface>
+                                <friction>
+                                        <mu>0.9</mu>
+                                        <mu2>0.9</mu2>
+                                </friction>
+                        </surface>
 		</collision>
 		<inertial>
 			<xacro:zero_origin/>
-			<mass value="0.5"/>
+			<mass value="${wheel_mass}"/>
 			<inertia ixx='0.3' ixy='0' ixz='0' iyy='0.3' iyz='0' izz='0.5'/>
 		</inertial>
 	</link>
+	<joint name='caster_axis' type='continuous'>
+		<origin xyz='-${base_length/2 - caster_axis_offset} 0 0' rpy='0 0 0'/>
+		<axis xyz='0 0 1'/>
+		<parent link='chassis'/>
+		<child link='caster_body'/>
+	</joint>
 	<!--caster wheel -->
-	<joint name='caster_wheel' type='fixed'>
-		<origin xyz='-${base_length/2 - caster_offset} 0 -${base_lift - tire_diam/2}' rpy='0 0 0'/>
-		<parent link='chassis'/>
-		<child link='caster'/>
+        <link name='caster_body'>
+                <!-- No visual for now -->
+		<!-- Should probably have physics at least -->
+		<inertial>
+			<xacro:zero_origin/>
+			<mass value="0.2"/>
+			<inertia ixx='0.3' ixy='0' ixz='0' iyy='0.3' iyz='0' izz='0.1'/>
+		</inertial>
+        </link>
+	<joint name='caster_wheel_joint' type='continuous'>
+		<origin xyz='-${caster_trail} 0 -${base_lift - tire_diam/2}' rpy='-${PI/2} 0 0'/>
+		<axis xyz='0 0 1'/>
+		<parent link='caster_body'/>
+		<child link='caster_wheel'/>
 	</joint>
-	<link name='caster'>
-		<collision>
-			<origin xyz='0 0 0' rpy='0 0 0'/>
+	<link name='caster_wheel'>
+		<visual>
+			<xacro:zero_origin/>
 			<geometry>
-				<sphere radius='${tire_diam / 2}'/>
-			</geometry>
-		</collision>
-		<inertial>
-			<mass value="0.5"/>
-			<inertia ixx='0.3' ixy='0' ixz='0' iyy='0.3' iyz='0' izz='0.3'/>
-		</inertial>
-		<visual name='visual'>
-			<origin xyz='0 0 0' rpy='0 0 0'/>
-			<geometry>
-				<sphere radius='${tire_diam / 2}'/>
+				<cylinder radius='${tire_diam / 2}' length='${tire_width}'/>
 			</geometry>
 			<material name="black"/>
 		</visual>
+		<collision>
+			<xacro:zero_origin/>
+			<geometry>
+				<cylinder radius='${tire_diam / 2}' length='${tire_width}'/>
+			</geometry>
+                        <surface>
+                                <friction>
+                                        <mu>0.9</mu>
+                                        <mu2>0.3</mu2>
+                                </friction>
+                        </surface>
+		</collision>
+		<inertial>
+			<xacro:zero_origin/>
+			<mass value="${wheel_mass}"/>
+			<inertia ixx='0.3' ixy='0' ixz='0' iyy='0.3' iyz='0' izz='0.5'/>
+		</inertial>
 	</link>
 	<!-- LIDAR -->
