Commit message: Hardware Driver progress, renamed files
Driver files moved to better locations. Tests currently do not work.

File: rover_ws/src/rover/description/urdf/rover.ros2_control.xacro (robot description, xacro)
@@ -2,27 +2,53 @@
 <robot xmlns:xacro="http://www.ros.org/wiki/xacro">
   <!-- Copied from: https://github.com/ros-controls/ros2_control_demos/blob/master/example_2/description/ros2_control/diffbot.ros2_control.xacro -->
-  <xacro:macro name="diffbot_ros2_control" params="name use_gazebo:=^|false">
-    <ros2_control name="${name}" type="system">
+  <xacro:macro name="rover_ros2_control" params="name use_gazebo:=^|false">
+    <ros2_control name="${name}/DiffDrive" type="actuator">
       <hardware>
-	<xacro:if value="${use_gazebo}">
-	  <plugin>gz_ros2_control/GazeboSimSystem</plugin>
-	</xacro:if>
-	<xacro:unless value="${use_gazebo}">
-	  <!-- Replace this with my own hardware interfaces -->
-	  <plugin>ros2_control_demo_example_2/DiffBotSystemHardware</plugin>
-	  <param name="example_param_hw_start_duration_sec">0</param>
-	  <param name="example_param_hw_stop_duration_sec">3.0</param>
-	  <param name="example_param_hw_slowdown">100</param> <!-- Unsure what this is for-->
-	</xacro:unless>
+        <!-- plugin to use in sim mode -->
+        <xacro:if value="${use_gazebo}">
+          <plugin>rover_hardware/DiffDrive</plugin>
+        </xacro:if>
+        <!-- otherwise, in real bot mode. -->
+        <xacro:unless value="${use_gazebo}">
+          <plugin>rover_hardware/DiffDrive</plugin>
+          <!-- Additional params:
+          <param name="example_param_hw_start_duration_sec">0</param>
+          <param name="example_param_hw_stop_duration_sec">3.0</param>
+          <param name="example_param_hw_slowdown">100</param>
+          -->
+        </xacro:unless>
+      </hardware>
+      <!-- Only controls velocity of motors -->
+      <!-- TODO: Add PID to make sure this stays accurate? -->
+      <joint name="left_wheel_joint">
+        <command_interface name="velocity"/>
+      </joint>
+      <joint name="right_wheel_joint">
+        <command_interface name="velocity"/>
+      </joint>
+    </ros2_control>
+    <!-- Arduino Encoder parser -->
+    <ros2_control name="${name}/DiffDrive" type="sensor">
+      <hardware>
+        <!-- plugin to use in sim mode -->
+        <xacro:if value="${use_gazebo}">
+          <plugin>rover_hardware/DiffDrive</plugin>
+        </xacro:if>
+        <!-- otherwise, in real bot mode. -->
+        <xacro:unless value="${use_gazebo}">
+          <plugin>rover_hardware/DiffDrive</plugin>
+          <!-- Additional params:
+            <param name="example_param_hw_start_duration_sec">0</param>
+            <param name="example_param_hw_stop_duration_sec">3.0</param>
+          <param name="example_param_hw_slowdown">100</param> -->
+        </xacro:unless>
       </hardware>
       <joint name="left_wheel_joint">
-	<command_interface name="velocity"/>
-	<state_interface name="position"/>
-	<state_interface name="velocity"/>
+        <state_interface name="position"/>
+        <state_interface name="velocity"/>
       </joint>
       <joint name="right_wheel_joint">
-	<command_interface name="velocity"/>
-	<state_interface name="position"/>
-	<state_interface name="velocity"/>
+        <state_interface name="position"/>
+        <state_interface name="velocity"/>
       </joint>
       <joint name="caster_axis">
@@ -35,2 +61,10 @@
   </xacro:macro>
 </robot>
+<!--
+<joint name="caster_axis">
+  <state_interface name="position"/>
+</joint>
+<joint name="caster_wheel_joint">
+  <state_interface name="position"/>
+</joint>
+-->

Commit message: Refactor of diffdrive hardware and arduino code.
Based on Diffdrive_Arduino and RosArduinoBridge, with alterations for
the current motor driver, microcontroller and encoders.

File: rover_ws/src/rover/description/urdf/rover.ros2_control.xacro (robot description, xacro)
@@ -2,6 +2,6 @@
 <robot xmlns:xacro="http://www.ros.org/wiki/xacro">
   <!-- Copied from: https://github.com/ros-controls/ros2_control_demos/blob/master/example_2/description/ros2_control/diffbot.ros2_control.xacro -->
-  <xacro:macro name="rover_ros2_control" params="name use_gazebo:=^|false">
-    <ros2_control name="${name}/DiffDrive" type="actuator">
+  <xacro:macro name="rover_ros2_control" params="name use_gazebo:=^|false rw_rate:=30">
+    <ros2_control name="${name}/DiffDrive" type="system" rw_rate="${rw_rate}">
       <hardware>
         <!-- plugin to use in sim mode -->
@@ -12,49 +12,23 @@
         <xacro:unless value="${use_gazebo}">
           <plugin>rover_hardware/DiffDrive</plugin>
-          <!-- Additional params:
-          <param name="example_param_hw_start_duration_sec">0</param>
-          <param name="example_param_hw_stop_duration_sec">3.0</param>
-          <param name="example_param_hw_slowdown">100</param>
+          <param name="left_wheel_name">left_wheel_joint</param>
+          <param name ="right_wheel_name">right_wheel_joint</param>
+          <!--
+          <param name ="loop_rate">30</param>
+          <param name ="device">0</param>
+          <param name ="baud_rate">0</param>
+          <param name ="timeout">0</param>
           -->
         </xacro:unless>
       </hardware>
-      <!-- Only controls velocity of motors -->
-      <!-- TODO: Add PID to make sure this stays accurate? -->
       <joint name="left_wheel_joint">
         <command_interface name="velocity"/>
-      </joint>
-      <joint name="right_wheel_joint">
-        <command_interface name="velocity"/>
-      </joint>
-    </ros2_control>
-    <!-- Arduino Encoder parser -->
-    <ros2_control name="${name}/DiffDrive" type="sensor">
-      <hardware>
-        <!-- plugin to use in sim mode -->
-        <xacro:if value="${use_gazebo}">
-          <plugin>rover_hardware/DiffDrive</plugin>
-        </xacro:if>
-        <!-- otherwise, in real bot mode. -->
-        <xacro:unless value="${use_gazebo}">
-          <plugin>rover_hardware/DiffDrive</plugin>
-          <!-- Additional params:
-            <param name="example_param_hw_start_duration_sec">0</param>
-            <param name="example_param_hw_stop_duration_sec">3.0</param>
-          <param name="example_param_hw_slowdown">100</param> -->
-        </xacro:unless>
-      </hardware>
-      <joint name="left_wheel_joint">
         <state_interface name="position"/>
         <state_interface name="velocity"/>
       </joint>
       <joint name="right_wheel_joint">
+        <command_interface name="velocity"/>
         <state_interface name="position"/>
         <state_interface name="velocity"/>
-      </joint>
-      <joint name="caster_axis">
-        <state_interface name="position"/>
-      </joint>
-      <joint name="caster_wheel_joint">
-        <state_interface name="position"/>
       </joint>
     </ros2_control>
